File: kicad/eagle-8.kicad_pcb (KiCad board)
At the start: 4 copper layers, 127.1 x 98.7 mm, 87 parts, among them CN1 AM3 bracket, J1 SC242, J2 PGA387, J3 same as Vcore, J4 Slot 1 L2

Commit message: removed most of the inner layer traces
Parts:
- removed H1, H2, H3, H4: 6mm, MountingHole:MountingHole_6mm
- RN1, RN10, RN11, RN12, RN13, RN14, RN15, RN16, RN17, RN18, RN19, RN2, RN20, RN21, RN22, RN23, RN24, RN25, RN26, RN27, RN28, RN29, RN3, RN30, RN31, RN32, RN33, RN34, RN35, RN4, RN5, RN6, RN7, RN8, RN9: footprint Resistor_SMD:R_Array_Convex_4x0612 -> eagle-8:VTT array
- moved R3 3.47 mm to (127.6, 105.3), turned to 0 degrees
- moved RN30 0.12 mm to (167.5, 76.9)
- moved RN27 0.10 mm to (167.5, 80.7)
- moved RN5 0.09 mm to (167.5, 92.2)
- moved RN6 0.08 mm to (167.5, 92.2)
- moved RN35 0.06 mm to (167.5, 84.5)
- moved RN1 0.05 mm to (167.5, 80.8)
Connections:
- RN12 pad 4: /D25 -> /D29
- RN14 pad 1: /D24 -> /D20
- RN14 pad 2: /D20 -> /D16
- RN14 pad 3: /D16 -> /D19
- RN14 pad 4: /D19 -> /D24
- RN16 pad 7: /D29 -> /D25
- RN23 pad 5: /DEP2 -> /DEP4
- RN25 pad 5: /DEP3 -> /BPM1
- RN25 pad 6: /DEP5 -> /D62
- RN25 pad 7: /D62 -> /DEP6
- RN25 pad 8: /DEP4 -> /DEP1
- RN26 pad 5: /DEP6 -> /PRDY
- RN26 pad 6: /PRDY -> /RESET
- RN26 pad 7: /DEP1 -> /D58
- RN26 pad 8: /D58 -> /DEP2
- RN28 pad 5: /AERR -> /BP2
- RN28 pad 6: /BP2 -> /DEP0
- RN28 pad 7: /BP3 -> /BINIT
- RN32 pad 5: /RESET -> /AERR
- RN32 pad 6: /BINIT -> /BP3
- RN32 pad 7: /DEP0 -> /DEP3
- RN32 pad 8: /BPM1 -> /DEP5
Routing:
- net /RESET: track 126.4 -> 89.3 mm, vias 1 -> 0
- net /D0: track 57.4 -> 36.8 mm
- net /D2: track 56.8 -> 36.9 mm
- net /BP3: track 90.0 -> 107.0 mm, vias 0 -> 1
- net /D1: track 53.8 -> 38.0 mm, vias 0 -> 1
- net /FRCERR: track 50.4 -> 35.3 mm
- net /D4: track 53.6 -> 39.6 mm
- net /THTRIP: track 78.4 -> 91.4 mm, vias 3 -> 0
- net /D3: track 51.9 -> 39.3 mm, vias 0 -> 1
- net /D6: track 50.7 -> 38.1 mm
- net /PRDY: track 110.6 -> 99.6 mm, vias 0 -> 1
- net /DEP5: track 80.1 -> 90.2 mm, vias 0 -> 1
- net /D25: track 59.4 -> 49.6 mm
- net /D5: track 49.2 -> 39.7 mm, vias 0 -> 1
- net /PICCLK: track 74.2 -> 82.9 mm
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- added copper zone on In2.Cu, net GND
- added copper zone on In1.Cu, net Vcore
- removed copper zone on In1.Cu, net GND
- removed copper zone on In2.Cu, net Vcore

Commit message: finalized routing
Parts:
- removed the C35 at (164.3, 55.2)
- removed J3: same as Vcore, Connector_PinHeader_2.54mm:PinHeader_2x04_P2.54mm_Vertical
- removed J4: Slot 1 L2, Connector_PinHeader_2.54mm:PinHeader_2x04_P2.54mm_Vertical
- added H1: MountingHole, MountingHole:MountingHole_3.2mm_M3_DIN965, F.Cu at (94.7, 86.2)
- added H2: MountingHole, MountingHole:MountingHole_3.2mm_M3_DIN965, F.Cu at (215.7, 86.2)
- C22, C23, C32, C33, C34: moved to F.Cu
- moved REF** 101.7 mm to (210.4, 105.4)
- moved G*** 95.9 mm to (207.6, 73.5)
- moved C35 41.4 mm to (198.6, 108.7)
- moved C36 37.2 mm to (206.8, 116.1), turned to 180 degrees
- moved C13 27.1 mm to (164.5, 68.9), turned to -90 degrees
- moved C32 17.9 mm to (164.7, 55.5)
- moved C11 16.2 mm to (163.6, 85.0), turned to 0 degrees
- moved C12 16.1 mm to (163.8, 81.5), turned to 0 degrees
- moved C21 14.7 mm to (162.8, 47.8)
- moved C19 12.6 mm to (158.6, 47.8)
- moved C30 11.9 mm to (148.5, 55.5)
- moved C14 10.5 mm to (148.1, 47.9)
- moved C29 8.38 mm to (148.2, 48.1)
- moved C31 8.09 mm to (143.5, 55.5)
- moved C8 7.64 mm to (163.7, 96.0)
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- renumbered C36 to C35, C37 to C36
Connections:
- C24 pad 2: VccS -> Vcore
- C25 pad 2: VccS -> Vcore
- C26 pad 2: VccS -> Vcore
- C27 pad 2: VccS -> Vcore
- C28 pad 2: VccS -> Vcore
- C29 pad 2: VccS -> Vcore
- C35 pad 1: VccS -> Vcore
- C36 pad 1: VccS -> Vcore
- J1 pad B113: VccL2 -> unconnected-(J1D-VCC_L2-PadB113)_1
- J1 pad B117: VccL2 -> unconnected-(J1D-VCC_L2-PadB113)
- J1 pad B121: VccL2 -> unconnected-(J1D-VCC_L2-PadB113)_2
- J2 pad AU1: VccS -> Vcore
- J2 pad AU39: VccS -> Vcore
- J2 pad AU43: VccS -> Vcore
- J2 pad AU47: VccS -> Vcore
- J2 pad AU5: VccS -> Vcore
- J2 pad AU9: VccS -> Vcore
- J2 pad AW3: VccS -> Vcore
- J2 pad AW41: VccS -> Vcore
- J2 pad AW45: VccS -> Vcore
- J2 pad AW7: VccS -> Vcore
- J2 pad AY1: VccS -> Vcore
- J2 pad AY3: VccS -> Vcore
- J2 pad AY39: VccS -> Vcore
- J2 pad AY41: VccS -> Vcore
- J2 pad AY43: VccS -> Vcore
- J2 pad AY45: VccS -> Vcore
- J2 pad AY47: VccS -> Vcore
- J2 pad AY5: VccS -> Vcore
- J2 pad AY7: VccS -> Vcore
- J2 pad AY9: VccS -> Vcore
- J2 pad BA3: VccS -> Vcore
- J2 pad BA41: VccS -> Vcore
- J2 pad BA45: VccS -> Vcore
- J2 pad BA7: VccS -> Vcore
- J2 pad BC19: VccS -> Vcore
- J2 pad BC23: VccS -> Vcore
- J2 pad BC27: VccS -> Vcore
- J2 pad BC31: VccS -> Vcore
- RN14 pad 4: /D24 -> /D25
- RN16 pad 6: /D26 -> /D24
- RN16 pad 7: /D25 -> /D26
- RN18 pad 5: /D44 -> /D45
- RN20 pad 5: /D49 -> /D52
- RN20 pad 6: /D52 -> /D51
- RN20 pad 7: /D51 -> /D42
- RN20 pad 8: /D45 -> /D44
- RN21 pad 8: /D42 -> /D49
- RN27 pad 5: /REQ2 -> /TRDY
- RN27 pad 6: /TRDY -> /REQ2
- RN35 pad 5: /RSP -> /AP0
- RN35 pad 6: /BR3 -> /RSP
- RN35 pad 7: /AP0 -> /BR3
Routing:
- net /AP1: track 83.8 -> 143.6 mm, vias 1 -> 4
- net /RSP: track 86.7 -> 142.1 mm, vias 1 -> 4
- net /AP0: track 91.8 -> 145.1 mm, vias 1 -> 3
- net GND: track 125.4 -> 97.6 mm
- net Net-(J2D-VREF0): track 168.4 -> 185.5 mm
- net VccL2: track 14.3 -> 0.00 mm, vias 3 -> 0
- net /D25: track 49.6 -> 61.8 mm
- net /RP: track 99.7 -> 108.5 mm
- net Vcore: track 48.5 -> 54.9 mm, vias 19 -> 33
- net /SMI: track 138.4 -> 132.8 mm
- net /D24: track 63.1 -> 67.7 mm
- net /D42: track 78.2 -> 74.2 mm, vias 3 -> 2
- net /D44: track 68.0 -> 71.1 mm
- net /D45: track 72.6 -> 69.9 mm
- net /A34: track 52.0 -> 50.1 mm
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- added copper zone on F.Cu, net Vcore
- removed copper zone on F.Cu, net VccL2
- removed copper zone on F.Cu, net VccS
Other:
- board text removed: "Do NOT insert jumpers into both headers at the same time!"
- board text removed: "L2 voltage"
