File: kicad/eagle-8.kicad_sch (KiCad schematic)
At the start: 64 parts, among them J1 SC242, J2 PGA387

Commit message: more improvements
Parts:
- removed C14, C15, C16, C17: 1000uF, Capacitor_THT:CP_Radial_D10.0mm_P5.00mm, symbol Device:C_Polarized
- removed H1, H2, H3, H4: 5.5mm, MountingHole:MountingHole_5.5mm, symbol Mechanical:MountingHole
- removed R4: 0, Resistor_SMD:R_0805_2012Metric, symbol Device:R
- removed R7, R8: 1K, Resistor_SMD:R_0805_2012Metric, symbol Device:R
- added C14, C15, C16, C17, C18, C19, C20, C21, C22, C23, C24, C25, C26, C27, C28, C29: 100n, Capacitor_SMD:C_0805_2012Metric, symbol Device:C_Small
- added C30, C31, C32, C33, C34, C35, C36, C37: 47uF, Capacitor_Tantalum_SMD:CP_EIA-7343-40_Kemet-Y_HandSolder, symbol Device:C_Polarized_Small
- added CN1: AM3 bracket, eagle-8:AM3 bracket, symbol eagle-8:AM3_bracket
- added J3: same as Vcore, Connector_PinHeader_2.54mm:PinHeader_2x04_P2.54mm_Vertical, symbol Connector_Generic:Conn_02x04_Odd_Even
- added J4: Slot 1 L2, Connector_PinHeader_2.54mm:PinHeader_2x04_P2.54mm_Vertical, symbol Connector_Generic:Conn_02x04_Odd_Even
- added R14: 56R, Resistor_SMD:R_0805_2012Metric, symbol Device:R
- R1, R2: value 1K -> 150R
- R3: value 150R? -> 150R
Connections:
- net AERR: now also RN28.5 (R4.2); no longer RN30.6 (R3.2)
- net D10: now also RN11.4 (R4.1); no longer RN11.3 (R3.1)
- net D11: now also RN11.2 (R2.1); no longer RN11.1 (R1.1)
- net D12: now also RN10.1 (R1.1); no longer RN10.2 (R2.1)
- net D13: now also RN13.4 (R4.1); no longer RN13.3 (R3.1)
- net D14: now also RN10.2 (R2.1); no longer RN11.4 (R4.1)
- net D15: now also RN11.3 (R3.1); no longer RN10.1 (R1.1)
- net D16: now also RN14.3 (R3.1); no longer RN14.1 (R1.1)
- net D17: now also RN11.1 (R1.1); no longer RN11.2 (R2.1)
- net D18: now also RN13.3 (R3.1); no longer RN13.1 (R1.1)
- net D19: now also RN14.4 (R4.1); no longer RN14.2 (R2.1)
- net D20: now also RN14.2 (R2.1); no longer RN13.4 (R4.1)
- net D21: now also RN13.2 (R2.1); no longer RN16.5 (R4.2)
- net D22: now also RN13.1 (R1.1); no longer RN13.2 (R2.1)
- net D23: now also RN16.5 (R4.2); no longer RN12.4 (R4.1)
- net D24: now also RN14.1 (R1.1); no longer RN16.6 (R3.2)
- net D25: now also RN12.4 (R4.1); no longer RN16.7 (R2.2)
- net D26: now also RN16.6 (R3.2); no longer RN14.3 (R3.1)
- net D29: now also RN16.7 (R2.2); no longer RN14.4 (R4.1)
- net D31: now also RN16.8 (R1.2); no longer RN17.5 (R4.2)
- net D38: now also RN17.5 (R4.2); no longer RN16.8 (R1.2)
- net FRCERR: now also R14.1
- net GND: now also J2.AS39 (TESTLO), J2.AS41 (TESTLO), J2.AS43 (TESTLO), J2.AS45 (TESTLO), J2.BA13 (TESTLO), J2.BA15 (TESTLO), J2.BA33 (TESTLO), J2.BA37 (TESTLO), J2.BC13 (TESTLO), J2.BC15 (TESTLO), J2.BC33 (TESTLO), J2.BC37 (TESTLO), J2.C21 (TESTLO), C14.1, C15.1, C16.1, C17.1, C18.1, C19.1, C20.1, C21.1, C22.1, C23.1, C24.1, C25.1, C26.1, C27.1, C28.1, C29.1, C30.2, C31.2, C32.2, C33.2, C34.2, C35.2, C36.2, C37.2
- net HIT: now also RN30.5 (R4.2); no longer RN30.7 (R2.2)
- net LOCK: now also RN30.7 (R2.2); no longer RN30.8 (R1.2)
- net REQ0: now also RN27.8 (R1.2); no longer RN35.5 (R4.2)
- net REQ2: now also RN27.5 (R4.2); no longer RN27.7 (R2.2)
- net REQ3: now also RN30.8 (R1.2); no longer RN27.5 (R4.2)
- net REQ4: now also RN27.7 (R2.2); no longer RN27.8 (R1.2)
- net RSP: now also RN35.5 (R4.2); no longer RN35.6 (R3.2)
- net VTT: now also R1.1, R2.1, C30.1, C31.1, R14.2
- net VccL2: now also J4.2 (Pin_2), J4.4 (Pin_4), J4.6 (Pin_6), J4.8 (Pin_8); no longer J2.AU1 (VccS), J2.AU39 (VccS), J2.AU43 (VccS), J2.AU47 (VccS), J2.AU5 (VccS), J2.AU9 (VccS), J2.AW3 (VccS), J2.AW41 (VccS), J2.AW45 (VccS), J2.AW7 (VccS), J2.AY1 (VccS), J2.AY3 (VccS), J2.AY39 (VccS), J2.AY41 (VccS), J2.AY43 (VccS), J2.AY45 (VccS), J2.AY47 (VccS), J2.AY5 (VccS), J2.AY7 (VccS), J2.AY9 (VccS), J2.BA3 (VccS), J2.BA41 (VccS), J2.BA45 (VccS), J2.BA7 (VccS), J2.BC19 (VccS), J2.BC23 (VccS), J2.BC27 (VccS), J2.BC31 (VccS)
- net Vcore: now also J2.A23 (TESTHI), J2.A25 (TESTHI), J2.AE39 (TESTHI), C14.2, C15.2, C16.2, C17.2, C18.2, C19.2, C20.2, C21.2, C22.2, C23.2, C32.1, C33.1, C34.1, C35.1, J3.1 (Pin_1), J3.3 (Pin_3), J3.5 (Pin_5), J3.7 (Pin_7); no longer R1.1, R2.2
- net at R1.2: now also J2.A1 (VREF0), J2.A47 (VREF4), J2.AE47 (VREF5), J2.AG45 (VREF7), J2.C7 (VREF1), J2.S7 (VREF2), J2.U41 (VREF6), J2.Y7 (VREF3), R2.2, R3.1; no longer J2.AE39 (TESTHI)
- net BR2: now reaches J2.AA1 (BR2#)
- net BR2: now also RN30.6 (R3.2)
- net BR3: now reaches J2.U9 (BR3#)
- net BR3: now also RN35.6 (R3.2)
- new net VccS: C24.2, C25.2, C26.2, C27.2, C28.2, C29.2, C36.1, C37.1, J2.AU1 (VccS), J2.AU39 (VccS), J2.AU43 (VccS), J2.AU47 (VccS), J2.AU5 (VccS), J2.AU9 (VccS), J2.AW3 (VccS), J2.AW41 (VccS), J2.AW45 (VccS), J2.AW7 (VccS), J2.AY1 (VccS), J2.AY3 (VccS), J2.AY39 (VccS), J2.AY41 (VccS), J2.AY43 (VccS), J2.AY45 (VccS), J2.AY47 (VccS), J2.AY5 (VccS), J2.AY7 (VccS), J2.AY9 (VccS), J2.BA3 (VccS), J2.BA41 (VccS), J2.BA45 (VccS), J2.BA7 (VccS), J2.BC19 (VccS), J2.BC23 (VccS), J2.BC27 (VccS), J2.BC31 (VccS), J3.2 (Pin_2), J3.4 (Pin_4), J3.6 (Pin_6), J3.8 (Pin_8), J4.1 (Pin_1), J4.3 (Pin_3), J4.5 (Pin_5), J4.7 (Pin_7)
- no-connect marks 17 -> 14
Other:
- moved on the sheet: C10, C11, C12, C13, C2, C3, C4, C5, C6, C7, C8, C9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

Commit message: removed most of the inner layer traces
Parts:
- RN1, RN10, RN11, RN12, RN13, RN14, RN15, RN16, RN17, RN18, RN19, RN2, RN20, RN21, RN22, RN23, RN24, RN25, RN26, RN27, RN28, RN29, RN3, RN30, RN31, RN32, RN33, RN34, RN35, RN4, RN5, RN6, RN7, RN8, RN9: footprint Resistor_SMD:R_Array_Convex_4x0612 -> eagle-8:VTT array
Connections:
- net AERR: now also RN32.5 (R4.2); no longer RN28.5 (R4.2)
- net BINIT: now also RN28.7 (R2.2); no longer RN32.6 (R3.2)
- net BP2: now also RN28.5 (R4.2); no longer RN28.6 (R3.2)
- net BP3: now also RN32.6 (R3.2); no longer RN28.7 (R2.2)
- net BPM1: now also RN25.5 (R4.2); no longer RN32.8 (R1.2)
- net D16: now also RN14.2 (R2.1); no longer RN14.3 (R3.1)
- net D19: now also RN14.3 (R3.1); no longer RN14.4 (R4.1)
- net D20: now also RN14.1 (R1.1); no longer RN14.2 (R2.1)
- net D24: now also RN14.4 (R4.1); no longer RN14.1 (R1.1)
- net D25: now also RN16.7 (R2.2); no longer RN12.4 (R4.1)
- net D29: now also RN12.4 (R4.1); no longer RN16.7 (R2.2)
- net D58: now also RN26.7 (R2.2); no longer RN26.8 (R1.2)
- net D62: now also RN25.6 (R3.2); no longer RN25.7 (R2.2)
- net DEP0: now also RN28.6 (R3.2); no longer RN32.7 (R2.2)
- net DEP1: now also RN25.8 (R1.2); no longer RN26.7 (R2.2)
- net DEP2: now also RN26.8 (R1.2); no longer RN23.5 (R4.2)
- net DEP3: now also RN32.7 (R2.2); no longer RN25.5 (R4.2)
- net DEP4: now also RN23.5 (R4.2); no longer RN25.8 (R1.2)
- net DEP5: now also RN32.8 (R1.2); no longer RN25.6 (R3.2)
- net DEP6: now also RN25.7 (R2.2); no longer RN26.5 (R4.2)
- net PRDY: now also RN26.5 (R4.2); no longer RN26.6 (R3.2)
- net RESET: now also RN26.6 (R3.2); no longer RN32.5 (R4.2)

Commit message: finalized routing
Parts:
- removed C35: 47uF, Capacitor_Tantalum_SMD:CP_EIA-7343-40_Kemet-Y_HandSolder, symbol Device:C_Polarized_Small
- removed J3: same as Vcore, Connector_PinHeader_2.54mm:PinHeader_2x04_P2.54mm_Vertical, symbol Connector_Generic:Conn_02x04_Odd_Even
- removed J4: Slot 1 L2, Connector_PinHeader_2.54mm:PinHeader_2x04_P2.54mm_Vertical, symbol Connector_Generic:Conn_02x04_Odd_Even
- added H1, H2: MountingHole, MountingHole:MountingHole_3.2mm_M3_DIN965, symbol Mechanical:MountingHole
- renumbered C36 to C35, C37 to C36
Connections:
- net VccS is gone; now on net Vcore: C24.2, C25.2, C26.2, C27.2, C28.2, C29.2, C35.1, C36.1, J2.AU1 (VccS), J2.AU39 (VccS), J2.AU43 (VccS), J2.AU47 (VccS), J2.AU5 (VccS), J2.AU9 (VccS), J2.AW3 (VccS), J2.AW41 (VccS), J2.AW45 (VccS), J2.AW7 (VccS), J2.AY1 (VccS), J2.AY3 (VccS), J2.AY39 (VccS), J2.AY41 (VccS), J2.AY43 (VccS), J2.AY45 (VccS), J2.AY47 (VccS), J2.AY5 (VccS), J2.AY7 (VccS), J2.AY9 (VccS), J2.BA3 (VccS), J2.BA41 (VccS), J2.BA45 (VccS), J2.BA7 (VccS), J2.BC19 (VccS), J2.BC23 (VccS), J2.BC27 (VccS), J2.BC31 (VccS)
- net AP0: now also RN35.5 (R4.2); no longer RN35.7 (R2.2)
- net BR3: now also RN35.7 (R2.2); no longer RN35.6 (R3.2)
- net D24: now also RN16.6 (R3.2); no longer RN14.4 (R4.1)
- net D25: now also RN14.4 (R4.1); no longer RN16.7 (R2.2)
- net D26: now also RN16.7 (R2.2); no longer RN16.6 (R3.2)
- net D42: now also RN20.7 (R2.2); no longer RN21.8 (R1.2)
- net D44: now also RN20.8 (R1.2); no longer RN18.5 (R4.2)
- net D45: now also RN18.5 (R4.2); no longer RN20.8 (R1.2)
- net D49: now also RN21.8 (R1.2); no longer RN20.5 (R4.2)
- net D51: now also RN20.6 (R3.2); no longer RN20.7 (R2.2)
- net D52: now also RN20.5 (R4.2); no longer RN20.6 (R3.2)
- net REQ2: now also RN27.6 (R3.2); no longer RN27.5 (R4.2)
- net RSP: now also RN35.6 (R3.2); no longer RN35.5 (R4.2)
- net TRDY: now also RN27.5 (R4.2); no longer RN27.6 (R3.2)
- net VccL2: no longer names the net of J1.B113 (VCC_L2), J1.B117 (VCC_L2), J1.B121 (VCC_L2)
- no-connect marks 14 -> 15
Other:
- moved on the sheet: C24, C25, C26, C27, C28, C29, C35, C36
